Commit message: Improve robot model and simulation for perfect operation
URDF Improvements:
- Increased base mass (35→40kg) and wheel mass (2.5→3kg) for better stability
- Added proper friction and damping properties to all links
- Enhanced differential drive plugin with velocity/acceleration limits
- Added joint damping for smoother motion
- Improved caster wheel physics with proper mass and damping
- Added forward-facing camera sensor for visualization
- Enhanced IMU sensor with realistic noise characteristics
- Removed invalid gz_frame_id elements (replaced with proper SDF config)

World File Improvements:
- Replaced failing Fuel actor with static worker model box
- Eliminates 404 errors and improves simulation reliability

Bridge Configuration:
- Added camera topics (image_raw, camera_info) for complete sensor suite

Launch Configuration:
- Increased spawn height (0.05→0.1m) to avoid ground collision
- Added allow_renaming flag for cleaner entity management

Testing Results:
- Simulation launches without warnings (gz_frame_id errors resolved)
- Fuel actor loading errors eliminated
- Lidar sensor working correctly (detecting obstacles at various ranges)
- IMU sensor working correctly (gravity detection, realistic noise)
- Differential drive functioning properly (odometry updating)
- Camera sensor configured and bridged to ROS 2
- All sensors publishing data correctly

File: ros2/src/safety_core_sim/description/agv.urdf.xacro (robot description, xacro)
@@ -7,9 +7,9 @@
   <xacro:property name="base_width"      value="0.60"/>
   <xacro:property name="base_height"     value="0.20"/>
-  <xacro:property name="base_mass"       value="35.0"/>
+  <xacro:property name="base_mass"       value="40.0"/>
   <xacro:property name="wheel_radius"    value="0.10"/>
   <xacro:property name="wheel_length"    value="0.05"/>
   <xacro:property name="wheel_separation" value="0.50"/>
-  <xacro:property name="wheel_mass"      value="2.5"/>
+  <xacro:property name="wheel_mass"      value="3.0"/>
   <xacro:property name="caster_radius"   value="0.04"/>
   <xacro:property name="lidar_height"    value="0.06"/>
@@ -69,4 +69,14 @@
     <xacro:box_inertia m="${base_mass}" x="${base_length}" y="${base_width}" z="${base_height}"/>
   </link>
+  <!-- Gazebo material properties for base -->
+  <gazebo reference="base_link">
+    <material>Gazebo/Grey</material>
+    <mu1>0.3</mu1>
+    <mu2>0.3</mu2>
+    <kp>1000000.0</kp>
+    <kd>100.0</kd>
+    <minDepth>0.001</minDepth>
+    <maxVel>0.01</maxVel>
+  </gazebo>
   <!-- ========================================================
        Drive wheels (left + right)
@@ -90,8 +100,28 @@
       <origin xyz="0 ${y_sign*wheel_separation/2.0} 0" rpy="0 0 0"/>
       <axis xyz="0 1 0"/>
+      <dynamics damping="0.1" friction="0.0"/>
     </joint>
   </xacro:macro>
   <xacro:drive_wheel prefix="left"  y_sign="1.0"/>
   <xacro:drive_wheel prefix="right" y_sign="-1.0"/>
+  <!-- Gazebo material properties for wheels -->
+  <gazebo reference="left_wheel_link">
+    <mu1>1.0</mu1>
+    <mu2>1.0</mu2>
+    <kp>1000000.0</kp>
+    <kd>100.0</kd>
+    <minDepth>0.001</minDepth>
+    <maxVel>0.01</maxVel>
+    <fdir1>0 1 0</fdir1>
+  </gazebo>
+  <gazebo reference="right_wheel_link">
+    <mu1>1.0</mu1>
+    <mu2>1.0</mu2>
+    <kp>1000000.0</kp>
+    <kd>100.0</kd>
+    <minDepth>0.001</minDepth>
+    <maxVel>0.01</maxVel>
+    <fdir1>0 1 0</fdir1>
+  </gazebo>
   <!-- ========================================================
        Caster (front + rear) for stability
@@ -100,11 +130,13 @@
     <link name="${prefix}_caster_link">
       <visual>
+        <origin xyz="0 0 0" rpy="0 0 0"/>
         <geometry><sphere radius="${caster_radius}"/></geometry>
         <material name="rubber_dark"><color rgba="0.1 0.1 0.1 1.0"/></material>
       </visual>
       <collision>
+        <origin xyz="0 0 0" rpy="0 0 0"/>
         <geometry><sphere radius="${caster_radius}"/></geometry>
       </collision>
-      <xacro:sphere_inertia m="0.3" r="${caster_radius}"/>
+      <xacro:sphere_inertia m="0.5" r="${caster_radius}"/>
     </link>
     <joint name="${prefix}_caster_joint" type="fixed">
@@ -112,8 +144,26 @@
       <child link="${prefix}_caster_link"/>
       <origin xyz="${x_sign*(base_length/2.0 - caster_radius)} 0 ${-(wheel_radius - caster_radius)}" rpy="0 0 0"/>
+      <dynamics damping="0.1" friction="0.0"/>
     </joint>
   </xacro:macro>
   <xacro:caster prefix="front" x_sign="1.0"/>
   <xacro:caster prefix="rear"  x_sign="-1.0"/>
+  <!-- Gazebo material properties for casters -->
+  <gazebo reference="front_caster_link">
+    <mu1>0.5</mu1>
+    <mu2>0.5</mu2>
+    <kp>1000000.0</kp>
+    <kd>100.0</kd>
+    <minDepth>0.001</minDepth>
+    <maxVel>0.01</maxVel>
+  </gazebo>
+  <gazebo reference="rear_caster_link">
+    <mu1>0.5</mu1>
+    <mu2>0.5</mu2>
+    <kp>1000000.0</kp>
+    <kd>100.0</kd>
+    <minDepth>0.001</minDepth>
+    <maxVel>0.01</maxVel>
+  </gazebo>
   <!-- ========================================================
        Lidar (planar, forward-mounted)
@@ -149,4 +199,22 @@
   </joint>
   <!-- ========================================================
+       Camera (forward-facing for visualization)
+  ======================================================== -->
+  <link name="camera_link">
+    <visual>
+      <geometry><box size="0.04 0.04 0.04"/></geometry>
+      <material name="camera_grey"><color rgba="0.3 0.3 0.3 1.0"/></material>
+    </visual>
+    <collision>
+      <geometry><box size="0.04 0.04 0.04"/></geometry>
+    </collision>
+    <xacro:box_inertia m="0.1" x="0.04" y="0.04" z="0.04"/>
+  </link>
+  <joint name="camera_joint" type="fixed">
+    <parent link="base_link"/>
+    <child link="camera_link"/>
+    <origin xyz="${lidar_x_offset} 0 ${base_height + 0.15}" rpy="0 0.3 0"/>
+  </joint>
+  <!-- ========================================================
        Gazebo plugins (Harmonic / gz-sim 8)
   ======================================================== -->
@@ -158,5 +226,9 @@
       <wheel_separation>${wheel_separation}</wheel_separation>
       <wheel_radius>${wheel_radius}</wheel_radius>
-      <max_linear_acceleration>1.0</max_linear_acceleration>
+      <max_linear_acceleration>2.0</max_linear_acceleration>
+      <max_linear_velocity>1.5</max_linear_velocity>
+      <max_angular_velocity>2.0</max_angular_velocity>
+      <min_wheel_torque>5.0</min_wheel_torque>
+      <max_wheel_torque>20.0</max_wheel_torque>
       <topic>/cmd_vel</topic>
       <odom_topic>/odom</odom_topic>
@@ -165,4 +237,5 @@
       <child_frame_id>base_footprint</child_frame_id>
       <odom_publish_frequency>50</odom_publish_frequency>
+      <enable_ros2_control>false</enable_ros2_control>
     </plugin>
   </gazebo>
@@ -179,5 +252,4 @@
       <topic>/scan</topic>
       <update_rate>15</update_rate>
-      <gz_frame_id>lidar_link</gz_frame_id>
       <ray>
         <scan>
@@ -214,8 +286,71 @@
     <sensor name="imu" type="imu">
       <topic>/imu</topic>
-      <gz_frame_id>imu_link</gz_frame_id>
       <update_rate>100</update_rate>
       <always_on>1</always_on>
+      <imu>
+        <angular_velocity>
+          <x>
+            <noise type="gaussian">
+              <mean>0.0</mean>
+              <stddev>0.0001</stddev>
+            </noise>
+          </x>
+          <y>
+            <noise type="gaussian">
+              <mean>0.0</mean>
+              <stddev>0.0001</stddev>
+            </noise>
+          </y>
+          <z>
+            <noise type="gaussian">
+              <mean>0.0</mean>
+              <stddev>0.0001</stddev>
+            </noise>
+          </z>
+        </angular_velocity>
+        <linear_acceleration>
+          <x>
+            <noise type="gaussian">
+              <mean>0.0</mean>
+              <stddev>0.001</stddev>
+            </noise>
+          </x>
+          <y>
+            <noise type="gaussian">
+              <mean>0.0</mean>
+              <stddev>0.001</stddev>
+            </noise>
+          </y>
+          <z>
+            <noise type="gaussian">
+              <mean>0.0</mean>
+              <stddev>0.001</stddev>
+            </noise>
+          </z>
+        </linear_acceleration>
+      </imu>
     </sensor>
   </gazebo>
+  <!-- Camera sensor -->
+  <gazebo reference="camera_link">
+    <sensor name="camera" type="camera">
+      <pose>0 0 0 0 0 0</pose>
+      <topic>/camera/image_raw</topic>
+      <update_rate>30</update_rate>
+      <camera>
+        <horizontal_fov>1.047</horizontal_fov>
+        <image>
+          <width>640</width>
+          <height>480</height>
+          <format>R8G8B8</format>
+        </image>
+        <clip>
+          <near>0.1</near>
+          <far>100.0</far>
+        </clip>
+      </camera>
+      <always_on>1</always_on>
+      <visualize>true</visualize>
+    </sensor>
+  </gazebo>
 </robot>

Commit message: Add EKF + navsat_transform localization stack with GPS outlier rejection
- New ekf_config.yaml: two-EKF + navsat_transform pattern (odom-frame +
  map-frame), tuned diagonal process noise, Mahalanobis-gated GPS odometry.
- New launch files: localization.launch.py (standalone bench/bag), safety_sim.launch.py.
- Updated agv_warehouse.launch.py: ekf:=true now spins up local EKF +
  navsat_transform_node + global EKF; gates GPS branch with gps:= arg.
- New diagnostics script test_localization.py: sensor liveness, fusion Hz,
  drift, GPS spike monitor (3sigma residual), TF availability.
- New nav2_params_odometry.yaml: AMCL/map_server-free Nav2 config used by
  the wheel-odometry default mode.
- New RViz configs: safety_simple.rviz, agv_nav2_robot_frame.rviz.
- Doc: ros2/LOCALIZATION.md (architecture, tuning, failure modes).
- Robot URDF: GPS link + Gazebo navsat sensor; ros_gz_bridge: /gps NavSatFix.
- safety_only.launch.py now optionally launches RViz with safety_simple.rviz.

File: ros2/src/safety_core_sim/description/agv.urdf.xacro (robot description, xacro)
@@ -197,4 +197,24 @@
     <child link="imu_link"/>
     <origin xyz="0 0 ${base_height + 0.02}" rpy="0 0 0"/>
+  </joint>
+  <!-- ========================================================
+       GPS (antenna on top of robot for localization)
+  ======================================================== -->
+  <link name="gps_link">
+    <visual>
+      <origin xyz="0 0 0" rpy="0 0 0"/>
+      <geometry><box size="0.08 0.08 0.02"/></geometry>
+      <material name="gps_black"><color rgba="0.1 0.1 0.1 1.0"/></material>
+    </visual>
+    <collision>
+      <origin xyz="0 0 0" rpy="0 0 0"/>
+      <geometry><box size="0.08 0.08 0.02"/></geometry>
+    </collision>
+    <xacro:box_inertia m="0.1" x="0.08" y="0.08" z="0.02"/>
+  </link>
+  <joint name="gps_joint" type="fixed">
+    <parent link="base_link"/>
+    <child link="gps_link"/>
+    <origin xyz="${lidar_x_offset} 0.05 ${base_height + 0.25}" rpy="0 0 0"/>
   </joint>
   <!-- ========================================================
@@ -354,3 +374,21 @@
     </sensor>
   </gazebo>
+  <!-- GPS sensor -->
+  <gazebo reference="gps_link">
+    <sensor name="gps" type="navsat">
+      <pose>0 0 0 0 0 0</pose>
+      <topic>/gps</topic>
+      <update_rate>10</update_rate>
+      <always_on>1</always_on>
+      <navsat>
+        <position_reference_frame_id>world</position_reference_frame_id>
+        <velocity_reference_frame_id>world</velocity_reference_frame_id>
+      </navsat>
+      <noise>
+        <type>gaussian</type>
+        <mean>0.0</mean>
+        <stddev>1.0</stddev>
+      </noise>
+    </sensor>
+  </gazebo>
 </robot>
